File: kicad_files/STEP.kicad_sch (KiCad schematic)
At the start: 73 parts, among them J1 CONN_MAG_01x03, J2 CONN_MAG_01x04, J3 CONN_MAG_01x09, Q1 AOCA32116E, Q2 SSM3K35CTC, Q3 SSM3K35CTC, U1 LSM6DSO32TR, U2 BQ297xy, U3 LM3671TL-1V8/NOPB, U4 STM32WB55CEU6TR, U5 ANT016008LCS2442MA2, U6 PKMCS0909E4000-R1, Y1 NX1612SA-32.000MHZ-CHP-CIS-3

Commit message: finished v0.9 schematic and layout, annotated for review
Parts:
- removed J1: CONN_MAG_01x03, symbol step_symbols_main:CONN_MAG_01x03
- removed J2: CONN_MAG_01x04, symbol step_symbols_main:CONN_MAG_01x04
- removed J3: CONN_MAG_01x09, symbol step_symbols_main:CONN_MAG_01x09
- removed R6, R7, R8, R9: R_10K, Resistor_SMD:R_0402_1005Metric, symbol ring-rescue:R_200K-step
- removed TP10, TP11, TP12, TP13, TP14, TP15, TP16, TP17, TP18, TP9, TP? (x2): Test_Point_SMD, TestPoint:TestPoint_Pad_1.0x1.0mm, symbol ring-rescue:Test_Point_SMD-step
- removed U?: LM3671TL-1V8/NOPB, symbol step_symbols_main:LM3671TL-1V8/NOPB
- added C16: C_YF, Capacitor_SMD:C_0402_1005Metric, symbol ring-rescue:C_100nF-step
- added C17: C_XF, Capacitor_SMD:C_0402_1005Metric, symbol ring-rescue:C_100nF-step
- added J1: CONN_FFC_FPC_VERT_8POS_0.5MM_SMD, step_footprints:tbf, symbol step_symbols_main:CONN_FFC_FPC_VERT_8POS_0.5MM_SMD
- added U7: LM3671TL-ADJ/NOPB, step_footprints:SOT-23-5, symbol step_symbols_main:LM3671TL-ADJ/NOPB
- AE1: footprint step-footprints:MLPF-WB55-01E3 -> step_footprints:MLPF-WB55-01E3
- Q1: footprint step-footprints:AOCA32116E -> step_footprints:AOCA32116E
- Q2, Q3: footprint (none) -> Package_TO_SOT_SMD:SOT-883
- R13, R15: renamed from R?; value R_10k -> R_200k
- R14, R16: renamed from R?; value R_X -> R_100k
- R17: renamed from R?; value R_10k -> R_Y
- TP3, TP4, TP5, TP6, TP7, TP8: footprint TestPoint:TestPoint_Pad_1.0x1.0mm -> TestPoint:TestPoint_Pad_D1.0mm
- U1: footprint step-footprints:LSM6DSO32TR -> step_footprints:LSM6DSO32TR
- U3: footprint (none) -> step_footprints:SOT-23-5
- U4: footprint step-footprints:QFN50P700X700X60-49N -> step_footprints:QFN50P700X700X60-49N
- U5: footprint step-footprints:ANT016008LCS2442MA2 -> step_footprints:ANT016008LCS2442MA2
- U6: footprint (none) -> step_footprints:SPKR_PKMCS0909E4000-R1
- U8: renamed from U?; footprint (none) -> step_footprints:SPKR_PKMCS0909E4000-R1
- Y1: footprint step-footprints:OSCSC105P160X120X35-4N -> step_footprints:OSCSC105P160X120X35-4N
- gave numbers to parts that had none: 4
Connections:
- net LED_1 is gone; now on net LED_DEBUG: D1.2 (A)
- net +1V8: now also U3.4 (FB), J1.1; no longer C18.1, L2.2, R17.2, U3.C3 (FB)
- net +BATT: now also U3.1 (VIN), U7.1 (VIN); no longer U3.A1 (VIN), U6.1
- net ADC_IN_0: now also J1.3
- net ADC_IN_1: now also J1.5
- net ADC_IN_2: now also J1.4
- net ADC_IN_3: now also J1.8
- net GND: now also U3.2 (GND), C17.2, J1.2, U7.2 (GND); no longer U3.A3 (GND)
- net LSM_INT1: now also U4.47 (PB7); no longer U4.46 (PB6)
- net LSM_INT2: now also U4.46 (PB6); no longer U4.29 (PB1)
- net VEN_AUX: now reaches R13.1, R14.2
- net VEN_AUX: now also U7.3 (EN)
- net RF_FILT: now reaches AE1.1 (OUT), U5.4 (Feed_point)
- net VSW_1V8: now reaches L1.1
- net VSW_1V8: now also U3.5 (SW); no longer U3.B2 (SW)
- net VEN_1V8: now reaches R15.1, R16.2
- net VEN_1V8: now also U3.3 (EN); no longer U3.C1 (EN)
- net AUX_BUZZER_DRAIN: now reaches Q3.3 (D), U6.2
- net VSW_AUX: now reaches L2.1
- net VSW_AUX: now also U7.5 (SW)
- net VFB_AUX: now reaches R17.1, R18.2
- net VFB_AUX: now also C16.2, C17.1, U7.4 (FB)
- net XTAL_FILT3: now reaches C8.1, U4.24 (OSC_OUT), Y1.3
- net BATT_BUZZER_DRAIN: now reaches Q2.3 (D), U8.2
- net XTAL_FILT1: now reaches C6.1, U4.25 (OSC_IN), Y1.1
- net LED_DEBUG: now reaches U4.37 (PA11)
- net BATT_FILT: now reaches C2.1, R1.1, U2.5 (BAT)
- net V_SENSE-: now reaches R2.2, U2.6 (V-)
- net BTN_0 renamed DIO_0
- net DIO_0: now also J1.6
- net BTN_1 renamed DIO_1
- net DIO_1: now also J1.7
- net BTN_2: no longer names the net of U4.16 (PA7)
- net BTN_3: no longer names the net of U4.17 (PA8)
- net BTN_4: no longer names the net of U4.18 (PA9)
- net C_gate renamed C_GATE
- net D_gate renamed D_GATE
- new net VAUX: C16.1, C18.1, L2.2, R17.2, U6.1
- no-connect marks 17 -> 19
Other:
- note added: "2:1 Resistor Divider to uC ADC. Vout = Vin/3"
- note added: "32MHz External clk; required for RF Layout note: minimize trace length between XTAL and uC. Maximize distance to BLE antenna"
- note added: "ADC Breakouts 4x ADC pins that can be used for either AIN/DIO"
- note added: "ADJ variant on fixed 1.8V buck"
- note added: "Accelerometer Interface SPI configuration. Consider switching to I2C in future for easier layout"
- note added: "Auxiliary Power: DNP unless voltage levels outside of default are needed"
- note added: "Bridge V[ZZ]SMPS pins for internal LDO config ref: page 27 on datasheet"
- note added: "Debug LED populate as needed"
- note added: "Ext Peripheral Interface"
- note added: "External XTAL trim caps. DNP, as likely unneeded"
- note added: "Extra DIO, likely unneeded"
- note added: "Feedback Network Cap stuffing for increased loop stability as needed"
- note added: "Firmware Note: any pins set-up as DIN will need internal pull-up/down configured on microcontroller"
- note added: "For JTAG programming interface"
- note added: "Haptic Feedback Interface"
- note added: "Intentionally 3.xV external haptic coin Vmin = 2V"
- note added: "Layout Note: Superimpose both footprints to minimize board footprint. Only 1 (if any) of the SMT piezo elements should be populated - in the best interest of maximizing battery capacity"
- note added: "Layout note: duplicate layout of both bucks"
- note added: "Layout note: use trace width of 0.2934mm Layout note: copy antenna design and shape from Datasheet"
- note added: "Low Side Drivers for haptics/pizeo buzzers"
- note added: "Low side shared drain NMOS Load Switch Bi-directional for charge/discharge cases"
- note added: "Pogo pin copper"
- note added: "RF Interface - BLE"
- note added: "Separate 0201 RF Decoupling Cap Layout Note: Route close to pin 23"
- note added: "System Power: Default to 1.8V, 600mA current limit; likely limiting factor is copper rather than buck. Exercise caution with high power peripherals Typ. Frequency @ 2MHz"
- note added: "VEN pin shall dip under 1V to disable buck converter when battery is discharged to 3V (corresponds to ~93% DoD)"
- note removed: "1/3 Resistor Divider to uC ADC"
- note removed: "32MHz External clk; required for RF Minimize trace length"
- note removed: "5x Button TP's - Solder N/O Button between 1V8 & it's pad"
- note removed: "ADC Breakout"
- note removed: "ADC Breakouts"
- note removed: "Backside LED for testing | DNP"
- note removed: "Button Breakout"
- note removed: "For Dial/Joystick compatibility || ADC2/ADC3 pins have DNP divider pads"
- note removed: "Haptic Feedback"
- note removed: "Intentionally 3.xV haptic coin Vmin = 2V"
- note removed: "Internal Pull -Down in SW"
- note removed: "JTAG Programming - Use in conjunction with Power connector"
- note removed: "Low side shared drain NMOS Load Switch"
- note removed: "Magnetic Connectors"
- note removed: "Peripherals - Use in conjunction with Power connector"
- note removed: "Power"
- note removed: "RF"
- note removed: "Separate 0201 RF Decoupling Cap Minimize length to pin 23"
- note removed: "Test Points & LEDs"
- note removed: "Variable output (DIFFERENT PN from fixed 1.8V)"
- note removed: "uC Power Wired for internal LDO config; see pg 27"
- company: (none) -> STEP
- title: (none) -> STEP Haptics + Controller 
- moved on the sheet: AE1, C1, C10, C11, C12, C13, C14, C15, C18, C2, C3, C4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

Commit message: post design review feedback, switching to external antenna for prototyping
Parts:
- removed J1: CONN_FFC_FPC_VERT_8POS_0.5MM_SMD, step_footprints:tbf, symbol step_symbols_main:CONN_FFC_FPC_VERT_8POS_0.5MM_SMD
- removed TP4, TP5, TP6, TP7, TP8: Test_Point_SMD, TestPoint:TestPoint_Pad_D1.0mm, symbol ring-rescue:Test_Point_SMD-step
- removed U5: ANT016008LCS2442MA2, step_footprints:ANT016008LCS2442MA2, symbol ring-rescue:ANT016008LCS2442MA2-step
- added C19, C20: C_XF, Capacitor_SMD:C_0402_1005Metric, symbol ring-rescue:C_100nF-step
- added J1: Molex_FFC_FPC_VERT_8POS_0.5MM_SMD_0525590853, step_footprints:tbf, symbol step_symbols_main:Molex_FFC_FPC_VERT_8POS_0.5MM_SMD_0525590853
- added J2: TC2030-IDC-TAGCONNECT, step_footprints:TAG_TC2030-IDC-NL, symbol step_symbols_main:TC2030-IDC-TAGCONNECT
- added R6: R_0, Jumper:SolderJumper-2_P1.3mm_Open_TrianglePad1.0x1.5mm, symbol STEP_Symbols:R_0
- added R7, R9: R_10K, Resistor_SMD:R_0402_1005Metric, symbol ring-rescue:R_200K-step
- added R8: R_10K, Resistor_SMD:R_0402_1005Metric, symbol ring-rescue:R_1K-step
- added U5: Molex_Conn_uFL_0734120110, Connector_Coaxial:U.FL_Molex_MCRF_73412-0110_Vertical, symbol step_symbols_main:Molex_Conn_uFL_0734120110
Connections:
- net +1V8: now also J1.1, J2.1 (VCC), R6.2, R8.2; no longer C5.1, L1.2, U3.4 (FB)
- net +BATT: now also R7.2
- net ADC_IN_0: now also U4.11 (PA2), J1.3; no longer U4.10 (PA1)
- net ADC_IN_1: now also U4.10 (PA1), J1.5; no longer U4.11 (PA2)
- net ADC_IN_2: now also J1.4
- net ADC_IN_3: now also J1.8
- net AUX_BUZZER_DRAIN: now also R9.1
- net BATT_BUZZER_DRAIN: now also R7.1
- net BOOT0: now also TP3.1
- net DIO_0: now also J1.6
- net DIO_1: now also J1.7
- net GND: now also C19.2, C20.2, J1.2, J2.5 (GND), U5.2 (GND)
- net NRST: now also J2.3 (nRESET), R8.1; no longer TP3.1
- net RF_FILT: now also U5.1 (RF)
- net SCK: now also J2.6 (SWO/TDO)
- net SWCLK: now also J2.4 (SWCLK/TCK)
- net SWDIO: now also J2.2 (SWDIO/TMS)
- net VAUX: now also R9.2
- net VEN_1V8: now also C20.1
- net VEN_AUX: now also C19.1
- new net VFB_1V8: C5.1, L1.2, R6.1, U3.4 (FB)
- no-connect marks 19 -> 15
Other:
- note added: "For external buttons/sensors"
- note added: "JTAG Interface"
- note added: "Layout note: use trace width of 0.2934mm Layout note: maintain 50ohm line impedance"
- note added: "SCK pin doubles as SWO"
- note added: "uFL Connector for external antenna"
- note removed: "Layout note: use trace width of 0.2934mm Layout note: copy antenna design and shape from Datasheet"
- note removed: "Pogo pin copper"
- note removed: "SMD Chip Antenna"
- moved on the sheet: AE1, C7, D1, Q2, Q3, R11, R12, R5, TP3, U6, U8
