File: board_rev2/espboard/espboard.kicad_pcb (KiCad board)
At the start: 2 copper layers, 38 x 66.1 mm, 48 parts, among them J1 ANO_SCROLL_WHEEL, J2 CONN_MAG_01x03, J3 TC2030-IDC-TAGCONNECT, Q1 AOCA32116E, SW1 SW_Push, SW2 SW_Push, SW3 SW_Push, SW4 SW_Push, U1 ESP32-PICO-MINI-02, U2 LM3671TL-ADJ/NOPB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

Commit message: ready for review
Parts:
- added JP1: SolderJumper_2_Open, Jumper:SolderJumper-2_P1.3mm_Open_RoundedPad1.0x1.5mm, F.Cu at (156.2, 82.8)
- added TP3: TestPoint, TestPoint:TestPoint_Pad_1.5x1.5mm, F.Cu at (166.0, 75.6)
- added kibuzzard-643F0A06: G***, kibuzzard-643F0A06, F.Cu at (166.0, 73.8)
- added kibuzzard-643F0B26: G***, kibuzzard-643F0B26, F.Cu at (156.2, 84.8)
- added kibuzzard-643F0B2D: G***, kibuzzard-643F0B2D, F.Cu at (156.2, 80.8)
- C1, C2, C3, C4, C5, C6, C7, C8, C9: footprint step:C_0603_1608Metric -> Capacitor_SMD:C_0603_1608Metric
- R1, R10, R11, R12, R13, R14, R15, R16, R17, R18, R19, R2, R20, R21, R3, R4, R5, R6, R7, R8, R9: footprint step:R_0603_1608Metric -> Resistor_SMD:R_0603_1608Metric
- moved L1 1.68 mm to (158.7, 83.5), turned to 90 degrees
- moved R3 1.61 mm to (152.8, 94.0)
- moved C3 1.54 mm to (154.3, 94.0)
- moved D1 1.35 mm to (163.8, 97.3)
- moved R21 1.35 mm to (163.8, 95.6)
- moved kibuzzard-643EF399 1.35 mm to (163.8, 98.9)
Connections:
- C4 pad 1: +3V3 -> Net-(C4-Pad1)
- C8 pad 1: +3V3 -> Net-(C4-Pad1)
- L1 pad 2: +3V3 -> Net-(C4-Pad1)
- R11 pad 1: +3V3 -> Net-(C4-Pad1)
Routing:
- net Net-(C4-Pad1): track 0.00 -> 19.8 mm
- net +3V3: track 68.1 -> 63.5 mm, vias 2 -> 0
- net Net-(L1-Pad1): track 7.60 -> 3.92 mm
- net GND: track 69.9 -> 71.5 mm
- net Net-(R21-Pad2): track 20.6 -> 19.2 mm, vias 4 -> 2
- net /DIAL_SW4: track 47.4 -> 48.3 mm
- net +BATT: track 35.9 -> 36.8 mm
