File: board_rev2/espboard/espboard.kicad_sch (KiCad schematic)
At the start: 36 parts, among them J1 ANO_SCROLL_WHEEL, J2 CONN_MAG_01x04, J3 TC2030-IDC-TAGCONNECT, Q1 AOCA32116E, U1 LM3671TL-ADJ/NOPB, U2 ESP32-S3-WROOM-1-N8, U3 BQ297xy

Commit message: layout rev done
Parts:
- removed C2: C_22uF, symbol Device:C
- removed C3: C_.1uF, symbol Device:C
- removed J2: CONN_MAG_01x04, symbol step:CONN_MAG_01x04
- removed U2: ESP32-S3-WROOM-1-N8, step:ESP32-S3-WROOM-1-N8, symbol step:ESP32-S3-WROOM-1-N8
- added C6: C_22uF, step:C_0603_1608Metric, symbol Device:C
- added C7: C_.1uF, step:C_0603_1608Metric, symbol Device:C
- added D1: LED, step:LED_0805_OEM, symbol Device:LED
- added J2: CONN_MAG_01x03, step:CONN_MAG_1x03, symbol step:CONN_MAG_01x03
- added R10, R2, R5, R6, R7, R8, R9: R_10k, step:R_0603_1608Metric, symbol Device:R
- added R21: R_200, step:R_0603_1608Metric, symbol Device:R
- added U1: ESP32-PICO-MINI-02, MODULE_ESP32-PICO-MINI-02, symbol step:ESP32-PICO-MINI-02
- C1: renamed from C4; footprint (none) -> step:C_0603_1608Metric
- C2: renamed from C1; footprint (none) -> step:C_0603_1608Metric
- C3: renamed from C5; footprint (none) -> step:C_0603_1608Metric
- C4: renamed from C6; footprint (none) -> step:C_0603_1608Metric
- C5: renamed from C7; footprint (none) -> step:C_0603_1608Metric
- C9: footprint Capacitor_SMD:C_0402_1005Metric -> step:C_0603_1608Metric; symbol ring-rescue:C_0.1uF-step -> Device:C
- J1: footprint (none) -> step:ANO_SCROLL_WHEEL
- J3: footprint (none) -> step:TAG_TC2030-IDC-NL
- L1: footprint (none) -> Inductor_SMD:L_0805_2012Metric_Pad1.15x1.40mm_HandSolder
- Q1: footprint step_footprints:AOCA32116E -> step:AOCA32116E
- R1: renamed from R3; footprint (none) -> step:R_0603_1608Metric
- R12: renamed from R5; footprint (none) -> step:R_0603_1608Metric
- R13, R14, R15, R16: renamed from R?; footprint (none) -> step:R_0603_1608Metric
- R17: renamed from R10; footprint Resistor_SMD:R_0402_1005Metric -> step:R_0603_1608Metric; symbol ring-rescue:R_330-step -> Device:R
- R18: renamed from R11; footprint Resistor_SMD:R_0402_1005Metric -> step:R_0603_1608Metric; symbol ring-rescue:R_2.2K-step -> Device:R
- R19: renamed from R12; footprint Resistor_SMD:R_0402_1005Metric -> step:R_0603_1608Metric; symbol ring-rescue:R_200K-step -> Device:R
- R20: renamed from R13; footprint Resistor_SMD:R_0402_1005Metric -> step:R_0603_1608Metric; symbol ring-rescue:R_100K-step -> Device:R
- R3: renamed from R1; footprint (none) -> step:R_0603_1608Metric
- R4: renamed from R2; footprint (none) -> step:R_0603_1608Metric
- SW1, SW2, SW3, SW4: renamed from SW?; footprint (none) -> Button_Switch_THT:SW_PUSH_6mm
- TP1, TP2: symbol ring-rescue:Test_Point_SMD-step -> Connector:TestPoint
- U2: renamed from U1; footprint (none) -> Package_TO_SOT_SMD:SOT-23-5
- renumbered R4 to R11
Connections:
- net +3V3: now also C6.1, C7.1, R10.1, R2.1, R5.1, R6.1, R7.1, R8.1, R9.1, U1.3 (3V3); no longer J1.1 (ENCA)
- net +BATT: now also J2.2
- net BATT_LVL: now also U1.7 (I39)
- net BUTTON_1_SENSE: now also R13.1, SW1.2, U1.35 (IO21); no longer R14.1, SW2.2
- net BUTTON_2_SENSE: now also R14.1, SW2.2, U1.26 (IO20); no longer R13.1, SW1.2
- net BUTTON_3_SENSE: now also R15.1, SW3.2, U1.21 (IO15); no longer R16.1, SW4.2
- net BUTTON_4_SENSE: now also R16.1, SW4.2, U1.19 (IO12); no longer R15.1, SW3.2
- net DIAL_ENCA: now also R2.2, U1.33 (IO19)
- net DIAL_ENCB: now also R5.2, U1.28 (IO8)
- net DIAL_SW1: now also R6.2, U1.27 (IO7)
- net DIAL_SW2: now also R7.2, U1.29 (IO5)
- net DIAL_SW3: now also R8.2, U1.34 (IO22)
- net DIAL_SW4: now also R9.2, U1.20 (IO13)
- net DIAL_SW5: now also R10.2, U1.18 (IO14)
- net ESP_EN: now also U1.8 (EN)
- net ESP_IO0: now also U1.23 (IO0)
- net ESP_RX: now also U1.30 (RXD0)
- net ESP_TX: now also U1.31 (TXD0)
- net GND: now also J1.8 (COMA), J1.9 (COMB), C6.2, C7.2, D1.1 (K), J2.1, J2.3, U1.1 (GND), U1.11 (GND), U1.14 (GND), U1.2 (GND), U1.36 (GND), U1.37 (GND), U1.38 (GND), U1.39 (GND), U1.40 (GND), U1.41 (GND), U1.42 (GND), U1.43 (GND), U1.44 (GND), U1.45 (GND), U1.46 (GND), U1.47 (GND), U1.48 (GND), U1.49 (GND), U1.50 (GND), U1.51 (GND), U1.52 (GND), U1.53 (GND), U1.54 (GND), U1.55 (GND), U1.56 (GND), U1.57 (GND), U1.58 (GND), U1.59 (GND), U1.60 (GND), U1.61 (GND); no longer J1.1 (ENCA)
- new net: D1.2 (A), R21.1
- new net: R21.2, U1.15 (IO25)
- new net: U1.25 (NC), U1.32 (NC)
- no-connect marks 21 -> 11
Other:
- note added: "ESP32-Pico SOC"
- note removed: "ESP32-Wroom SOC"
- moved on the sheet: C1, J1, R1, R13, R14, R15, R16, SW1, SW2, SW3, SW4

Commit message: ready for review
Parts:
- added JP1: SolderJumper_2_Open, Jumper:SolderJumper-2_P1.3mm_Open_RoundedPad1.0x1.5mm, symbol Jumper:SolderJumper_2_Open
- added TP3: TestPoint, TestPoint:TestPoint_Pad_1.5x1.5mm, symbol Connector:TestPoint
- C1, C2, C3, C4, C5, C6, C7, C8, C9: footprint step:C_0603_1608Metric -> Capacitor_SMD:C_0603_1608Metric
- R1, R10, R11, R12, R13, R14, R15, R16, R17, R18, R19, R2, R20, R21, R3, R4, R5, R6, R7, R8, R9: footprint step:R_0603_1608Metric -> Resistor_SMD:R_0603_1608Metric
- U1: footprint MODULE_ESP32-PICO-MINI-02 -> step:MODULE_ESP32-PICO-MINI-02
Connections:
- net +3V3: now also JP1.2 (B); no longer C4.1, C8.1, L1.2, R11.1
- net GND: now also TP3.1
- new net: C4.1, C8.1, JP1.1 (A), L1.2, R11.1
